Commit message: Update robot configuration files

File: my_robot_description/urdf/robot.gazebo.xacro (robot description, xacro)
@@ -1,4 +1,6 @@
 <?xml version="1.0"?>
 <robot xmlns:xacro="http://www.ros.org/wiki/xacro">
+    <xacro:property name="wheel_y_offset" value="0.15"/>
+    <xacro:property name="wheel_radius"   value="0.07"/>
     <gazebo>
         <plugin name="gz::sim::systems::DiffDrive" filename="gz-sim-diff-drive-system">

File: my_robot_description/urdf/robot.urdf.xacro (robot description, xacro)
@@ -1,5 +1,4 @@
 <?xml version="1.0"?>
 <robot name="my_robot" xmlns:xacro="http://www.ros.org/wiki/xacro">
-    <xacro:include filename="$(find my_robot_description)/urdf/robot.gazebo.xacro"/>
     <xacro:property name="base_length" value="0.3"/>
     <xacro:property name="base_width"  value="0.3"/>
@@ -16,5 +15,5 @@
     <xacro:property name="lidar_mass"   value="0.1"/>
     <xacro:property name="lidar_z_offset" value="0.13"/>
-    <xacro:property name="mesh_path" default="package://my_robot_description/meshes"/>
+    <xacro:property name="mesh_path" default="/root/workspaces/ros2_ws/src/task4-my_robot_description/my_robot_description/meshes"/>
     <xacro:property name="base_footprint_z" value="0.15"/>
     <link name="base_footprint"/>
@@ -45,5 +44,5 @@
     <link name="lidar_link">
         <visual>
-            <geometry><mesh filename="$(mesh_path)lidar.STL"/></geometry>
+            <geometry><mesh filename="$(dirname)/../meshes/lidar.STL"/></geometry>
             <material name="lidar_gray"><color rgba="0.5 0.5 0.5 1.0"/></material>
         </visual>
