Commit message: Import ros2-robot package

File: urdf/robot.urdf.xacro (robot description, xacro)
@@ -3,6 +3,7 @@
     <xacro:include filename="$(find ros2-robot)/urdf/robot.gazebo.xacro"/>
     <xacro:arg name="mesh_path" default="package://ros2-robot/meshes/"/>
-    <xacro:property name="base_radius" value="0.25"/>
-    <xacro:property name="base_length"  value="0.15"/>
+    <xacro:property name="base_width" value="0.20"/>
+    <xacro:property name="base_height" value="0.10"/>
+    <xacro:property name="base_length"  value="0.30"/>
     <xacro:property name="base_mass"   value="3.0"/>
     <xacro:property name="wheel_radius" value="0.05"/>
@@ -10,12 +11,23 @@
     <xacro:property name="wheel_mass"   value="0.5"/>
     <xacro:property name="wheel_x_offset" value="0.10"/>
-    <xacro:property name="wheel_y_offset" value="0.15"/>
-    <xacro:property name="wheel_z_offset" value="-0.08"/>
+    <xacro:property name="wheel_y_offset" value="0.075"/>
+    <xacro:property name="wheel_z_offset" value="-0.04"/>
     <xacro:property name="caster_radius" value="0.05"/>
     <xacro:property name="caster_mass" value="0.03"/>
+    <xacro:property name="caster_x_offset" value="0.06"/>
+     <xacro:property name="caster_y_offset" value="0.00"/>
+    <xacro:property name="caster_z_offset" value="-0.04"/>
     <xacro:property name="lidar_radius" value="0.06"/>
     <xacro:property name="lidar_length" value="0.04"/>
     <xacro:property name="lidar_mass"   value="0.1"/>
-    <xacro:property name="lidar_z_offset" value="0.13"/>
+    <xacro:property name="lidar_z_offset" value="0.07"/>
+    <xacro:property name="lidar_y_offset" value="0.00"/>
+    <xacro:property name="lidar_x_offset" value="0.07"/>
+    <xacro:property name="camera_size" value="0.06"/>
+    <xacro:property name="camera_height" value="0.04" />
+    <xacro:property name="camera_mass"  value="0.1"/>
+    <xacro:property name="camera_z_offset" value="0.02"/>
+    <xacro:property name="camera_y_offset" value="0.0"/>
+    <xacro:property name="camera_x_offset" value="0.18"/>
     <xacro:property name="base_footprint_z" value="0.15"/>
     <link name="base_footprint"/>
@@ -30,16 +42,16 @@
             <mass value="${base_mass}"/>
             <inertia
-               ixx="${(1/12) * base_mass * (3*base_radius*base_radius + base_length*base_length)}"
+               ixx="${(1/12) * base_mass * (base_width*base_width + base_height*base_height)}"
                     ixy="0.0" ixz="0.0"
-                    iyy="${(1/12) * base_mass * (3*base_radius*base_radius + base_length*base_length)}"
+                    iyy="${(1/12) * base_mass * (base_height*base_height + base_length*base_length)}"
                     iyz="0.0"
-                    izz="${(1/2) * base_mass * (base_radius*base_radius)}"/>
+                    izz="${(1/2) * base_mass * (base_width*base_width +  base_length*base_length)}"/>
         </inertial>
         <visual>
-            <geometry><cylinder radius="${base_radius}" length= "${base_length}"/></geometry>
+            <geometry><box size="${base_length} ${base_width} ${base_height}"/></geometry>
             <material name="chassis_color"><color rgba="0.4 0.5 0.3 1.0"/></material>
         </visual>
         <collision>
-            <geometry><cylinder radius="${base_radius}" length= "${base_length}"/></geometry>
+            <geometry><box size="${base_height} ${base_width} ${base_length}"/></geometry>
         </collision>
     </link>
@@ -60,5 +72,23 @@
         <parent link="base_link"/>
         <child link="lidar_link"/>
-        <origin xyz="0 0 ${lidar_z_offset}" rpy="0 0 0"/>
+        <origin xyz="${lidar_x_offset} ${lidar_y_offset} ${lidar_z_offset}" rpy="0 0 0"/>
+    </joint>
+    <link name="camera_link">
+        <visual>
+            <geometry><mesh filename="$(arg mesh_path)zed.stl"/></geometry>
+            <material name="camera_black"><color rgba="0 0 0 1.0"/></material>
+        </visual>
+        <collision>
+            <geometry><box size="${camera_size} ${camera_size} ${camera_height}"/></geometry>
+        </collision>
+        <inertial>
+            <mass value="${camera_mass}"/>
+            <inertia ixx="0.0001" ixy="0.0" ixz="0.0" iyy="0.0001" iyz="0.0" izz="0.0001"/>
+        </inertial>
+    </link>
+    <joint name="camera_joint" type="fixed">
+        <parent link="base_link"/>
+        <child link="camera_link"/>
+        <origin xyz="${camera_x_offset} ${camera_y_offset} ${camera_z_offset}" rpy="0 0 0"/>
     </joint>
     <xacro:macro name="wheel" params="prefix x_reflect y_reflect">
@@ -114,5 +144,5 @@
             <parent link="base_link"/>
             <child link="${prefix}_caster_link"/>
-            <origin xyz="${x_reflect * wheel_x_offset} ${y_reflect * wheel_y_offset} ${wheel_z_offset}" rpy="0 0 0"/>
+            <origin xyz="${x_reflect * caster_x_offset} ${y_reflect * caster_y_offset} ${caster_z_offset}" rpy="0 0 0"/>
             <axis xyz="0 1 0"/>
         </joint>

Commit message: Update URDF properties and geometry for camera and caster

File: urdf/robot.urdf.xacro (robot description, xacro)
@@ -16,5 +16,5 @@
     <xacro:property name="caster_mass" value="0.03"/>
     <xacro:property name="caster_x_offset" value="0.06"/>
-     <xacro:property name="caster_y_offset" value="0.00"/>
+    <xacro:property name="caster_y_offset" value="0.00"/>
     <xacro:property name="caster_z_offset" value="-0.04"/>
     <xacro:property name="lidar_radius" value="0.06"/>
@@ -53,5 +53,5 @@
         </visual>
         <collision>
-            <geometry><box size="${base_height} ${base_width} ${base_length}"/></geometry>
+            <geometry><box size="${base_length} ${base_width} ${base_height}"/></geometry>
         </collision>
     </link>
@@ -76,13 +76,24 @@
     <link name="camera_link">
         <visual>
-            <geometry><mesh filename="$(arg mesh_path)zed.stl"/></geometry>
-            <material name="camera_black"><color rgba="0 0 0 1.0"/></material>
+            <origin xyz="0 0 0" rpy="0 0 0"/>
+            <geometry>
+                <mesh filename="$(arg mesh_path)zed.stl"/>
+            </geometry>
+            <material name="camera_black">
+                <color rgba="0.5 0.5 0.5 1.0"/>
+            </material>
         </visual>
         <collision>
-            <geometry><box size="${camera_size} ${camera_size} ${camera_height}"/></geometry>
+            <origin xyz="0 0 0" rpy="0 0 0"/>
+            <geometry>
+                <box size="0.08 0.03 0.03"/>
+            </geometry>
         </collision>
         <inertial>
-            <mass value="${camera_mass}"/>
-            <inertia ixx="0.0001" ixy="0.0" ixz="0.0" iyy="0.0001" iyz="0.0" izz="0.0001"/>
+            <mass value="0.1"/>
+            <origin xyz="0 0 0" rpy="0 0 0"/>
+            <inertia ixx="0.00005" ixy="0.0" ixz="0.0"
+                     iyy="0.00005" iyz="0.0"
+                     izz="0.00005"/>
         </inertial>
     </link>
@@ -90,5 +101,11 @@
         <parent link="base_link"/>
         <child link="camera_link"/>
-        <origin xyz="${camera_x_offset} ${camera_y_offset} ${camera_z_offset}" rpy="0 0 0"/>
+        <origin xyz="0.3 0 0.08" rpy="0 0 0"/>
+    </joint>
+    <link name="camera_optical_link"/>
+    <joint name="camera_optical_joint" type="fixed">
+        <parent link="camera_link"/>
+        <child link="camera_optical_link"/>
+        <origin xyz="0 0 0" rpy="-1.5708 0 -1.5708"/>
     </joint>
     <xacro:macro name="wheel" params="prefix x_reflect y_reflect">
@@ -150,4 +167,4 @@
     <xacro:wheel prefix="left_front"  x_reflect="1"  y_reflect="1"/>
     <xacro:wheel prefix="right_front" x_reflect="1"  y_reflect="-1"/>
-    <xacro:caster_wheel prefix="rear" x_reflect="-1.2" y_reflect="0"/>
+    <xacro:caster_wheel prefix="rear" x_reflect="-1" y_reflect="0"/>
 </robot>

Commit message: Update robot.urdf.xacro

File: urdf/robot.urdf.xacro (robot description, xacro)
@@ -24,10 +24,9 @@
     <xacro:property name="lidar_y_offset" value="0.00"/>
     <xacro:property name="lidar_x_offset" value="0.07"/>
-    <xacro:property name="camera_size" value="0.06"/>
-    <xacro:property name="camera_height" value="0.04" />
+>
     <xacro:property name="camera_mass"  value="0.1"/>
     <xacro:property name="camera_z_offset" value="0.02"/>
     <xacro:property name="camera_y_offset" value="0.0"/>
-    <xacro:property name="camera_x_offset" value="0.18"/>
+    <xacro:property name="camera_x_offset" value="0.16"/>
     <xacro:property name="base_footprint_z" value="0.15"/>
     <link name="base_footprint"/>
@@ -87,9 +86,9 @@
             <origin xyz="0 0 0" rpy="0 0 0"/>
             <geometry>
-                <box size="0.08 0.03 0.03"/>
+                <box size="0.02 0.1 0.03"/>
             </geometry>
         </collision>
         <inertial>
-            <mass value="0.1"/>
+            <mass value="${caster_mass}"/>
             <origin xyz="0 0 0" rpy="0 0 0"/>
             <inertia ixx="0.00005" ixy="0.0" ixz="0.0"
@@ -101,5 +100,5 @@
         <parent link="base_link"/>
         <child link="camera_link"/>
-        <origin xyz="0.3 0 0.08" rpy="0 0 0"/>
+        <origin xyz="${camera_x_offset} ${camera_y_offset} ${camera_z_offset}" rpy="0 0 0"/>
     </joint>
     <link name="camera_optical_link"/>

Commit message: Update robot.urdf.xacro

File: urdf/robot.urdf.xacro (robot description, xacro)
@@ -27,5 +27,5 @@
     <xacro:property name="camera_z_offset" value="0.02"/>
     <xacro:property name="camera_y_offset" value="0.0"/>
-    <xacro:property name="camera_x_offset" value="0.16"/>
+    <xacro:property name="camera_x_offset" value="0.161"/>
     <xacro:property name="base_footprint_z" value="0.15"/>
     <link name="base_footprint"/>
